File: t-dsp_tac5212_audio_shield_adaptor.kicad_sch (KiCad schematic)
At the start: 212 parts, among them IC1 Logic Level Shifter - 74HCT2G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, J1 jumper, J10 JST-XH Connector, J11 JST-XH Connector, J12 RGB LED HEADEER, J13 Conn_01x02, J14 Conn_01x03, J15 Conn_01x01, J16 Conn_01x02, J17 Conn_02x04_Odd_Even, J18 Conn_02x02_Odd_Even, J19 Conn_01x01, J2 GROUND HEADER, J20 Conn_01x01, J21 jumper, J22 35RAPC4BV4, J23 35RAPC4BV4, J24 Conn_01x04, J25 PRT-14417, J26 73725-0110BLF, J27 Conn_01x04, J3 jumper, J4 jumper, J5 jumper, J6 jumper, J7 jumper, J8 PJRAS2X1S01X, J9 PJRAS2X1S01X, Q1 DMG2307L-7, Q2 DMG2307L-7, SW1 SW_SPST, SW2 TL1105WF160Q - 3.15mm actuator, SW3 SW_SPST, SW4 SW_SPST, SW5 RotaryEncoder_Switch_MP, SW6 TL1105WF160Q - 3.15mm actuator, SW7 TL1105WF160Q - 3.15mm actuator, SW8 TL1105WF160Q - 3.15mm actuator, T108 Tab, T109 Tab, T110 Tab, T111 Tab, U1 Teensy 4.1 - DEVKIT, U10 TPD4E02B04DQA, U2 ESP32-DevKitC - DEVKIT, U3 Power Mux & Protect - TPS2116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, U4 Optoisolators - H11L1SM - 6-S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, U5 Dual Buffer - SN74LVC2G125DCTR, U6 Dual Buffer - SN74LVC2G125DCTR, U7 Dual Buffer - SN74LVC2G125DCTR, U8 Dual Buffer - SN74LVC2G125DCTR, U9 Dual Buffer - 74HCT2G17GW,125

Commit message: Update t-dsp_tac5212_audio_shield_adaptor.kicad_sch
clean up BOM
Parts:
- J21, R12, USB_HOST_1, board_outline1: now not fitted; now left out of the parts list
- U1: now left out of the parts list
Connections:
- net at MIC2.4 (LRCLK-WS-FS): now also MIC1.4 (LRCLK-WS-FS)
- net at MIC1.4 (LRCLK-WS-FS): no longer MIC2.4 (LRCLK-WS-FS)
Changed lines of the file:
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@@
 		(unit 1)
 		(exclude_from_sim no)
-		(in_bom yes)
+		(in_bom no)
 		(on_board yes)
-		(dnp no)
+		(dnp yes)
 		(property "Reference" "R12"
 			(at -563.372 450.088 90)
@@
 		(unit 1)
 		(exclude_from_sim no)
-		(in_bom yes)
+		(in_bom no)
 		(on_board yes)
-		(dnp no)
+		(dnp yes)
 		(fields_autoplaced yes)
 		(property "Reference" "board_outline1"
@@
 		(unit 1)
 		(exclude_from_sim no)
-		(in_bom yes)
+		(in_bom no)
 		(on_board yes)
-		(dnp no)
+		(dnp yes)
 		(property "Reference" "J21"
 			(at -372.11 866.1399 90)
@@
 		(unit 1)
 		(exclude_from_sim no)
-		(in_bom yes)
+		(in_bom no)
 		(on_board yes)
 		(dnp yes)
@@
 		(unit 1)
 		(exclude_from_sim no)
-		(in_bom yes)
+		(in_bom no)
 		(on_board yes)
-		(dnp no)
+		(dnp yes)
 		(property "Reference" "USB_HOST_1"
 			(at 824.865 599.44 0)

Commit message: Add new components, 3D models, and update PCB layout
Add footprints and symbols for BLM15AG601SN1D, MSM261DGT003,
PESD5V0F1BL_315, 35RAPC4BV4, and passive 0402 components.
Add corresponding 3D models. Update schematic, PCB layout,
and existing footprints.
Parts:
- added D10, D11, D6, D7, D8, D9: ~, project_fp:PESD5V0F1BL_315, symbol Diode:1N4148
- added FB1, FB2, FB3, FB4, FB5, FB6: 600Ω@100MHz, project_fp:BLM15AG601SN1D, symbol Device:FerriteBead_Small
- added J28, J29: 35RAPC4BV4, project_fp:SWITCHCRAFT_35RAPC4BV4, symbol 35RAPC4BV4:35RAPC4BV4
- added R55, R56, R57: 49.9 ohm, project_fp:R_0402_1005Metric_Pad0.72x0.64mm_HandSolder, symbol Device:R_Small
- C1: footprint project_fp:C_0805_2012Metric_Pad1.15x1.40mm_HandSolder -> project_fp:C_0402_1005Metric_Pad0.74x0.62mm_HandSolder; LCSC C6119929 -> (none); LCSC_MPN CGA0805X7R105K500MT -> (none); LCSC_Manufacturer HRE -> (none); Package / Case C0805 -> (none)
- C10, C40: footprint project_fp:C_0805_2012Metric_Pad1.15x1.40mm_HandSolder -> project_fp:C_0402_1005Metric_Pad0.74x0.62mm_HandSolder; Package / Case C0805 -> (none)
- C7, C9, D3, USBA1: now not fitted
- HPTRS2: Label OUT -> IN
- MK1, MK2: value SPK0641HT4H-1 -> MSM261DGT003; footprint project_fp:SPK0641HT4H-1 -> project_fp:MSM261DGT003; symbol SPK0641HT4H-1:SPK0641HT4H-1 -> MSM261DGT003:MSM261DGT003; LCSC (none) -> C48227730; LCSC_MPN (none) -> MSM261DGT003; LCSC_Manufacturer (none) -> MEMS; Package / Case (none) -> LGA-6(2x4)
- R11: footprint project_fp:R_0805_2012Metric_Pad1.15x1.40mm_HandSolder -> project_fp:R_0402_1005Metric_Pad0.72x0.64mm_HandSolder; LCSC C17414 -> (none); LCSC_MPN 0805W8F1002T5E -> (none); LCSC_Manufacturer UNI-ROYAL -> (none); Package / Case R0805 -> (none)
- R13, R14: footprint project_fp:R_0805_2012Metric_Pad1.15x1.40mm_HandSolder -> project_fp:R_0402_1005Metric_Pad0.72x0.64mm_HandSolder; LCSC C17520 -> (none); LCSC_MPN 0805W8F2201T5E -> (none); LCSC_Manufacturer UNI-ROYAL -> (none); Package / Case R0805 -> (none)
- R3, R6, R9: footprint project_fp:R_0805_2012Metric_Pad1.15x1.40mm_HandSolder -> project_fp:R_0402_1005Metric_Pad0.72x0.64mm_HandSolder; LCSC C17720 -> C87044; LCSC_MPN 0805W8F499JT5E -> (none); LCSC_Manufacturer UNI-ROYAL -> (none); Package / Case R0805 -> (none)
Connections:
- net TEENSY_LED+ is gone; now on net TEENSY_LED: D3.1 (DIN), IC1.3 (2Y)
- net 3.3V: now also MK1.6 (SELECT), D6.2 (A), D7.2 (A), FB5.1, FB6.1; no longer MK1.3 (SELECT), MK1.4 (VDD), MK2.4 (VDD)
- net GND: now also MK1.2 (GND), MK2.2 (GND), D10.1 (K), D11.1 (K), D6.1 (K), D7.1 (K), D8.1 (K), D9.1 (K); no longer MK1.6 (GND), MK2.3 (SELECT)
- net GPIGPI1: now also R56.1, R57.1; no longer MK1.1 (DATA), MK2.1 (DATA)
- net GPIO1: now also FB3.2, FB4.2, R55.2; no longer MK1.2 (CLOCK), MK2.2 (CLOCK), board_outline1.40 (GPIO1)
- net at MIC2.4 (LRCLK-WS-FS): now also MIC1.4 (LRCLK-WS-FS)
- net at MIC1.4 (LRCLK-WS-FS): no longer MIC2.4 (LRCLK-WS-FS)
- new net: D8.2 (A), FB2.2, MK2.3 (DATA)
- new net: FB2.1, R56.2
- new net: D10.2 (A), FB3.1, MK2.4 (CLOCK)
- new net: FB1.1, R57.2
- new net: D9.2 (A), FB1.2, MK1.3 (DATA)
- new net: R55.1, board_outline1.40 (GPIO1)
- new net: FB6.2, MK2.1 (VDD)
- new net: D11.2 (A), FB4.1, MK1.4 (CLOCK)
- new net: FB5.2, MK1.1 (VDD)

Commit message: Fix ESD diode values and R13 value format for BOM correctness
Parts:
- C1: LCSC (none) -> C29266; LCSC_MPN (none) -> CL05A105KO5NNNC; LCSC_Manufacturer (none) -> Samsung Electro-Mechanics; Package / Case (none) -> 0402
- C10, C40: LCSC (none) -> C60474; LCSC TYPE (none) -> SMD; LCSC_MPN (none) -> CC0402KRX7R7BB104; LCSC_Manufacturer (none) -> YAGEO; Package / Case (none) -> 0402
- C36, C37, C39: Manufacturer Kyocera AVX -> (none); Manufacturer_Part_Number 08055C104M4T4A -> (none); mouser 581-08055C104M4T4A -> (none)
- C38: Manufacturer KEMET -> (none); Manufacturer_Part_Number C0805C104K5RAC7411 -> (none); mouser 80-C0805C104K5RACLR -> (none)
- D10, D11, D6, D7, D8, D9: value ~ -> ESD DIODE; LCSC TYPE (none) -> SMD; LCSC_MPN (none) -> PESD5V0F1BL,315; LCSC_Manufacturer (none) -> Nexperia; Package / Case (none) -> DFN1006-2
- ETHERNET1: Manufacturer WIZnet -> (none); Manufacturer_Part_Number J1B1211CCD -> (none); mouser 950-J1B1211CCD -> (none)
- ETHERNET_J1: Digikey - -> (none); Manufacturer - -> (none); Manufacturer_Part_Number - -> (none); mouser - -> (none)
- FB1, FB2, FB3, FB4, FB5, FB6: LCSC TYPE (none) -> SMD; LCSC_MPN (none) -> BLM15AG601SN1D; LCSC_Manufacturer (none) -> muRata; Package / Case (none) -> 0402
- G3: Digikey - -> (none); Manufacturer - -> (none); Manufacturer_Part_Number ~jumper -> (none); mouser - -> (none)
- HPTRS1, HPTRS2: Manufacturer Switchcraft -> (none); Manufacturer_Part_Number 35RAPC3BH3 -> (none)
- J22, J23, J28, J29: MANUFACTURER Switchcraft Inc. -> (none); MAXIMUM_PACKAGE_HIEGHT 12.573mm -> (none); PARTREV G -> (none); STANDARD Manufacturer Recommendations -> (none)
- J25: Availability In Stock -> (none); Check_prices https://www.snapeda.com/parts/PRT-14417/SparkFun/view-part/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 -> (none); Description_1 QWIIC JST CONNECTOR - SMD 4-PIN -> (none); MANUFACTURER SparkFun Electronics -> (none); MAXIMUM_PACKAGE_HEIGHT 2.9 mm -> (none); MF SparkFun Electronics -> (none); MP PRT-14417 -> (none); PARTREV NA -> (none); Price None -> (none); STANDARD Manufacturer Recommendations -> (none); SnapEDA_Link https://www.snapeda.com/parts/PRT-14417/SparkFun/view-part/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 -> (none)
- J26: Availability In Stock -> (none); Check_prices https://www.snapeda.com/parts/737250110BLF/Amphenol/view-pa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 -> (none); Description_1 USB, 2.0 TYPE A, RECEPTACLE, TH; USB Connector Type:USB Typ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 -> (none); MANUFACTURER AMPHENOL -> (none); MAXIMUM_PACKAGE_HEIGHT 15.03mm -> (none); MF Amphenol -> (none); MP 737250110BLF -> (none); PARTREV AL1 -> (none); Price None -> (none); SNAPEDA_PN 73725-0110BLF -> (none); STANDARD Manufacturer Recommendations -> (none); SnapEDA_Link https://www.snapeda.com/parts/737250110BLF/Amphenol/view-pa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 -> (none)
- J8, J9: Availability In Stock -> (none); Check_prices https://www.snapeda.com/parts/PJRAS2X1S01X/SWITCHCRAFT/view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 -> (none); Description_1 Connector, 2POS RA SHLD PHJK RE | Switchcraft PJRAS2X1S01X -> (none); MANUFACTURER Switchcraft -> (none); MF Switchcraft Inc. -> (none); MP PJRAS2X1S01X -> (none); Price None -> (none); SnapEDA_Link https://www.snapeda.com/parts/PJRAS2X1S01X/SWITCHCRAFT/view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 -> (none)
- MK1, MK2: Availability In Stock -> (none); Check_prices https://www.snapeda.com/parts/SPK0641HT4H-1/Knowles/view-pa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 -> (none); Description_1 20 Hz ~ 20 kHz Digital, PDM Microphone MEMS (Silicon) 1.6 V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 -> (none); LCSC TYPE (none) -> SMD; MANUFACTURER Knowles -> (none); MAXIMUM_PACKAGE_HEIGHT 1.1mm -> (none); MF Knowles -> (none); MP SPK0641HT4H-1 -> (none); PARTREV C -> (none); Price None -> (none); SNAPEDA_PN SPK0641HT4H-1 -> (none); STANDARD Manufacturer Recommendations -> (none); SnapEDA_Link https://www.snapeda.com/parts/SPK0641HT4H-1/Knowles/view-pa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 -> (none)
- Q1, Q2: Height 1.1 -> (none)
- R11: LCSC (none) -> C60490; LCSC_MPN (none) -> RC0402FR-0710KL; LCSC_Manufacturer (none) -> YAGEO; Package / Case (none) -> 0402
- R13, R14: value 2.21k ohm -> 2.21k; LCSC (none) -> C2906865; LCSC_MPN (none) -> FRC0402F2201TS; LCSC_Manufacturer (none) -> FOJAN; Package / Case (none) -> 0402
- R3, R6, R9: LCSC_MPN (none) -> RC0402FR-0749R9L; LCSC_Manufacturer (none) -> YAGEO; Package / Case (none) -> 0402
- R55, R56, R57: LCSC TYPE (none) -> SMD; LCSC_MPN (none) -> RC0402FR-0749R9L; LCSC_Manufacturer (none) -> YAGEO; Package / Case (none) -> 0402
- TR2: Manufacturer Everlight Electronics -> (none); Manufacturer_Part_Number FCR6842032R -> (none)
- TT2: Manufacturer Everlight Electronics -> (none); Manufacturer_Part_Number FCR6842032T -> (none)
Connections:
- net 3.3V: no longer D6.2 (A), D7.2 (A)
- net GND: no longer MK1.7 (GND), MK1.8 (GND), MK2.7 (GND), MK2.8 (GND)
- net at MIC2.4 (LRCLK-WS-FS): now also MIC1.4 (LRCLK-WS-FS)
- net at MIC1.4 (LRCLK-WS-FS): no longer MIC2.4 (LRCLK-WS-FS)
- net at FB6.2, MK2.1 (VDD): now also D7.2 (A)
- net at FB5.2, MK1.1 (VDD): now also D6.2 (A)
Other:
- moved on the sheet: C10, C40, FB5, FB6
